File: pcb/Capstone.kicad_sch (KiCad schematic)
At the start: 109 parts, among them IC1 HSFPAR004A, IC2 HSFPAR004A, IC3 HSFPAR004A, IC4 HSFPAR004A, J1 Conn_01x14_Socket, J2 Conn_01x14_Socket, J3 Conn_01x12_Socket, P1 USB_C_Plug_USB2.0, Q1 SS8050, Q2 SS8050, SW1 SW_Push, SW2 SW_Push, U1 ADS1015IDGS, U10 INA333xxDGK, U11 BMM350, U12 ICM-42688-P, U13 ICM-42688-P, U14 TLV75718PDBV, U2 ESP32-S3-WROOM-1, U3 TLV75733PDBV, U4 USBLC6-2SC6, U5 CP2102N-Axx-xQFN28, U6 INA333xxDGK, U7 ADS1015IDGS, U8 INA333xxDGK, U9 INA333xxDGK

Commit message: Connect components on PCB
Add electronic connections for printed circuit board components.
Parts:
- removed C40, C41: 0.1u, Capacitor_SMD:C_0603_1608Metric, symbol Device:C
- removed C42: 2.2u, Capacitor_SMD:C_0603_1608Metric, symbol Device:C
- removed J1: Conn_01x14_Socket, Connector_PinSocket_2.54mm:PinSocket_2x07_P2.54mm_Vertical, symbol Connector:Conn_01x14_Socket
- removed U11: BMM350, BMM350:BGA9_BMM350_BOS, symbol BMM350:BMM350
- added C43, C44: 10n, Capacitor_SMD:C_0603_1608Metric, symbol Device:C
- added J1: Conn_01x12_Socket, Connector_PinSocket_2.54mm:PinSocket_2x06_P2.54mm_Vertical, symbol Connector:Conn_01x12_Socket
- added J4: Conn_01x04_Socket, Connector_PinSocket_2.54mm:PinSocket_2x02_P2.54mm_Vertical, symbol Connector:Conn_01x04_Socket
Connections:
- net CS0: now also J3.8 (Pin_8), U2.22 (IO14); no longer J3.4 (Pin_4), U2.18 (IO10)
- net CS1: now also J1.5 (Pin_5)
- net EN: now also J1.1 (Pin_1)
- net GND: now also U14.4 (GND), U3.4 (GND), U4.2 (GND), C43.2, C44.2, J4.3 (Pin_3), J4.4 (Pin_4)
- net INT_IMU0: now also J3.4 (Pin_4), U2.18 (IO10); no longer J3.8 (Pin_8), U2.22 (IO14)
- net INT_IMU1: now also J1.12 (Pin_12)
- net INT_MAG1: now also J1.3 (Pin_3)
- net IO0: now also C7.2, SW1.2
- net IO1: now also R38.1; no longer C7.2, R36.1, SW1.2
- net IO17: now also R36.1, J1.10 (Pin_10); no longer R38.1
- net IO18: now also R37.1, J1.8 (Pin_8); no longer R39.1
- net IO2: now also R39.1; no longer R37.1
- net IO8: now also J1.6 (Pin_6)
- net SCK0: now also J3.7 (Pin_7), U2.21 (IO13); no longer J3.6 (Pin_6), U2.20 (IO12)
- net SCK1: now also J1.9 (Pin_9)
- net SDI0: now also J3.6 (Pin_6), U2.20 (IO12); no longer J3.5 (Pin_5), U2.19 (IO11)
- net SDI1: now also J1.7 (Pin_7)
- net SDO0: now also J3.5 (Pin_5), U2.19 (IO11); no longer J3.7 (Pin_7), U2.21 (IO13)
- net SDO1: now also J1.11 (Pin_11)
- net USB_D+: now also J1.2 (Pin_2)
- net USB_D-: now also J1.4 (Pin_4)
- net USB_D_N: now also U4.4 (I/O2); no longer U4.6 (I/O1)
- net USB_D_P: now also U4.6 (I/O1); no longer U4.4 (I/O2)
- net VBUS: now also C43.1, C44.1
- net VCC_1V8: now also J4.2 (Pin_2)
- net VCC_3V3: now also J4.1 (Pin_1)
- net F3_N: now reaches IC4.2 (V2), U10.2 (-)
- net F3_P: now reaches IC4.4 (V1), U10.3 (+)
- net USB_DI_N: now reaches P1.A7 (D-)
- net USB_DI_N: now also U4.3 (I/O2); no longer U4.1 (I/O1)
- net USB_DI_P: now reaches P1.A6 (D+)
- net USB_DI_P: now also U4.1 (I/O1); no longer U4.3 (I/O2)
- net F0_N: now reaches IC1.2 (V2), U6.2 (-)
- net F0_P: now reaches IC1.4 (V1), U6.3 (+)
- net F1_N: now reaches IC2.2 (V2), U8.2 (-)
- net F1_P: now reaches IC2.4 (V1), U8.3 (+)
- net F2_N: now reaches IC3.2 (V2), U9.2 (-)
- net F2_P: now reaches IC3.4 (V1), U9.3 (+)
Other:
- note added: "Power Connection for Breakout Boards"
- note removed: "Need specific cap check datasheet"
- moved on the sheet: D1, P1, U4

Commit message: Revise PCB for procurement
Revise printed circuit board with feedback from industry sponsor. Final design to send to JLCPCB.

 - Add Gerber files

 - Add Component Placement List and position files
Parts:
- removed C3: 4.7u, Capacitor_SMD:C_0603_1608Metric, symbol Device:C
- removed C36, C38: 10u, Capacitor_SMD:C_0603_1608Metric, symbol Device:C
- removed C37, C39, C4: 0.1u, Capacitor_SMD:C_0603_1608Metric, symbol Device:C
- removed J1, J3: Conn_01x12_Socket, Connector_PinSocket_2.54mm:PinSocket_2x06_P2.54mm_Vertical, symbol Connector:Conn_01x12_Socket
- removed J2: Conn_01x14_Socket, Connector_PinSocket_2.54mm:PinSocket_2x07_P2.54mm_Vertical, symbol Connector:Conn_01x14_Socket
- removed J4: Conn_01x04_Socket, Connector_PinSocket_2.54mm:PinSocket_2x02_P2.54mm_Vertical, symbol Connector:Conn_01x04_Socket
- removed P1: USB_C_Plug_USB2.0, Connector_USB:USB_C_Receptacle_HRO_TYPE-C-31-M-12, symbol Connector:USB_C_Plug_USB2.0
- removed Q1, Q2: SS8050, Package_TO_SOT_SMD:SOT-23, symbol Transistor_BJT:SS8050
- removed R29: 10k, Resistor_SMD:R_0603_1608Metric, symbol Device:R
- removed R30, R31: 4k7, Resistor_SMD:R_0603_1608Metric, symbol Device:R
- removed R34, R35: 5k1, Resistor_SMD:R_0603_1608Metric, symbol Device:R
- removed R7, R8: 0, Resistor_SMD:R_0603_1608Metric, symbol Device:R
- removed U14: TLV75718PDBV, Package_TO_SOT_SMD:SOT-23-5, symbol Regulator_Linear:TLV75718PDBV
- removed U5: CP2102N-Axx-xQFN28, Package_DFN_QFN:QFN-28-1EP_5x5mm_P0.5mm_EP3.35x3.35mm, symbol Interface_USB:CP2102N-Axx-xQFN28
- added D3: LED (AMBER), LED_SMD:LED_0603_1608Metric, symbol Device:LED
- added J1, J2, J3, J4: Conn_01x01, MountingHole:MountingHole_3.2mm_M3_DIN965_Pad, symbol Connector_Generic:Conn_01x01
- added J5: Conn_01x02, Connector_PinHeader_2.54mm:PinHeader_1x04_P2.54mm_Horizontal, symbol Connector_Generic:Conn_01x04
- added J6: USB_C_Receptacle, Connector_USB:USB_C_Receptacle_GCT_USB4105-xx-A_16P_TopMnt_Horizontal, symbol Connector:USB_C_Receptacle
- added J7: Conn_02x02_Counter_Clockwise, Connector_PinSocket_2.54mm:PinSocket_2x02_P2.54mm_Vertical, symbol Connector_Generic:Conn_02x02_Counter_Clockwise
- C31, C35: value 2.2u -> 2.2u +/- 10% X7R
- C32, C33: value 10n -> 10n +/- 10% X7R
- C9: value 10u -> 22u
- D1: value D_Schottky -> D_Schottky BAT760; footprint Diode_SMD:D_2114_3652Metric -> Diode_SMD:D_SOD-323F
- D2: value LED -> LED (RED)
- IC1, IC2, IC3, IC4: LCSC Part # (none) -> C470800; now not fitted
- R13, R17, R21, R25: value 499 -> 6.49k +/- 1%
- R14, R18, R22, R26: value 10k -> 10k +/- 1%
- R15, R19, R23, R27: value 3k -> 3k +/- 1%
- R2: value 22k1 -> 5.1k
- R3: value 47k5 -> 5.1k
- R36, R37, R38, R39: now not fitted
- R4: value 1k -> 10k
- R5: value 10k -> 100
- R6: value 10k -> 220
- SW1, SW2: footprint Button_Switch_SMD:SW_SPST_EVQQ2 -> Button_Switch_SMD:SW_SPST_EVQP7A
- U1, U7: LCSC Part # (none) -> C193969; Manufacturer_Name (none) -> TI; Manufacturer_Part_Number (none) -> ADS1015IDGSR
- U10, U6, U8, U9: LCSC Part # (none) -> C19450; Manufacturer_Name (none) -> TI; Manufacturer_Part_Number (none) -> INA333AIDGKR
- U12, U13: symbol ICM 42688-P:ICM-42688-P -> ICM_42688_P:ICM-42688-P; LCSC Part # (none) -> C1850418; Manufacturer_Name (none) -> TDK InvenSense; Manufacturer_Part_Number (none) -> ICM-42688-P
- U2: LCSC Part # (none) -> C2913197; Manufacturer_Name (none) -> ESPRESSIF; Manufacturer_Part_Number (none) -> ESP32-S3-WROOM-1-N4
- U3: LCSC Part # (none) -> C485517; Manufacturer_Name (none) -> TI; Manufacturer_Part_Number (none) -> TLV75733PDBVR
- U4: LCSC Part # (none) -> C7519; Manufacturer_Name (none) -> ST; Manufacturer_Part_Number (none) -> USBLC6-2SC6
Connections:
- net IO21 is gone; now on net EXT_BTN: U2.23 (IO21)
- net IO38 is gone; now on net EXT_LED: U2.31 (IO38)
- net IO8 is gone; now on net STATUS_LED: U2.12 (IO8)
- net IO9 is gone; now on net INT_IMU0: U2.17 (IO9)
- net USB_DI_N is gone; now on net USB_D_N: U4.3 (I/O2)
- net USB_DI_P is gone; now on net USB_D_P: U4.1 (I/O1)
- net GND: now also R2.2, R3.2, R4.2, U12.11 (RESV), U12.7 (RESV), U13.11 (RESV), U13.7 (RESV), D3.1 (K), J1.1 (Pin_1), J2.1 (Pin_1), J3.1 (Pin_1), J4.1 (Pin_1), J5.1 (Pin_1), J6.A1 (GND), J6.A12 (GND), J6.B1 (GND), J6.B12 (GND), J6.SH (SHIELD), J7.1 (Pin_1); no longer R3.1
- net INT_IMU0: no longer U2.18 (IO10)
- net INT_IMU1: now also U2.10 (IO17); no longer U2.9 (IO16)
- net RXD0: now also J5.3 (Pin_3)
- net SCL: now also R32.1, U2.24 (IO47); no longer R33.1, U2.25 (IO48)
- net SDA: now also R33.1, U2.25 (IO48); no longer R32.1, U2.24 (IO47)
- net TXD0: now also J5.2 (Pin_2)
- net USB_D+: now also U4.6 (I/O1), J6.A6 (D+), J6.B6 (D+); no longer U2.14 (USB_D+)
- net USB_D-: now also U4.4 (I/O2), J6.A7 (D-), J6.B7 (D-); no longer U2.13 (USB_D-)
- net USB_D_N: now also U2.13 (USB_D-); no longer U4.4 (I/O2)
- net USB_D_P: now also U2.14 (USB_D+); no longer U4.6 (I/O1)
- net VBUS: now also J6.A4 (VBUS), J6.A9 (VBUS), J6.B4 (VBUS), J6.B9 (VBUS); no longer R2.1
- net VCC_3V3: now also J5.4 (Pin_4), J7.2 (Pin_2); no longer R4.2
- net at R5.1: now also J7.4 (Pin_4)
- net STATUS_LED: now reaches R6.2
- net EXT_BTN: now reaches R4.1
- net EXT_BTN: now also J7.3 (Pin_3)
- net CS0: no longer names the net of U2.22 (IO14)
- net CS0: no longer U12.12 (AP_CS)
- net CS1 renamed CS_IMU1
- net CS_IMU1: now also U2.8 (IO15); no longer U2.5 (IO5)
- net DTR renamed EXT_LED
- net INT_MAG1 renamed F0_d
- net F0_d: now also R36.1
- net IO1 renamed F2_d
- net F2_d: now also U2.38 (IO2); no longer U2.39 (IO1)
- removed net IO17: R36.1, U2.10 (IO17)
- net IO18: no longer names the net of U2.11 (IO18)
- net IO18: no longer R37.1
- net IO2 renamed F3_d
- net F3_d: now also U2.39 (IO1); no longer U2.38 (IO2)
- net IO3: no longer names the net of U2.15 (IO3)
- net IO35: no longer names the net of U2.28 (IO35)
- net IO36: no longer names the net of U2.29 (IO36)
- net IO37: no longer names the net of U2.30 (IO37)
- net IO39: no longer names the net of U2.32 (IO39)
- net IO40: no longer names the net of U2.33 (IO40)
- net IO41: no longer names the net of U2.34 (IO41)
- net IO42: no longer names the net of U2.35 (IO42)
- net IO45: no longer names the net of U2.26 (IO45)
- net IO46: no longer names the net of U2.16 (IO46)
- net RTS: no longer names the net of R6.1
- net RTS: now also D3.2 (A)
- net SCK0 renamed CLK_IMU0
- net CLK_IMU0: now also U2.20 (IO12); no longer U2.21 (IO13)
- net SCK1 renamed CLK_IMU1
- net SDI0 renamed CONTROLLER_SDO_IMU0
- net CONTROLLER_SDO_IMU0: now also U2.19 (IO11); no longer U2.20 (IO12)
- net SDI1 renamed CONTROLLER_SDO_IMU1
- net SDO0 renamed CONTROLLER_SDI_IMU0
- net CONTROLLER_SDI_IMU0: now also U2.21 (IO13); no longer U2.19 (IO11)
- net SDO1 renamed CONTROLLER_SDI_IMU1
- net CONTROLLER_SDI_IMU1: now also U2.9 (IO16); no longer U2.8 (IO15)
- new net CC1: J6.A5 (CC1), R2.1
- new net CC2: J6.B5 (CC2), R3.1
- new net CS_IMU0: U12.12 (AP_CS), U2.18 (IO10)
- new net F1_d: R37.1, U2.5 (IO5)
- no-connect marks 18 -> 22
Other:
- note added: "Boot/Reset Buttons"
- note added: "External ADCs"
- note added: "External LED + Button header"
- note added: "Force sensors and amplifiers"
- note added: "GAIN = 16.4"
- note added: "IMUs"
- note added: "Internal ADC conn"
- note added: "Mounting holes"
- note added: "Power and Data I/O (USB, UART)"
- note added: "Reset"
- note removed: "GAIN = 200"
- note removed: "Is it necesssary to add series resistors and pull ups on SDI and SDO lines?"
- note removed: "Might want to use external crystal"
- note removed: "Power Connection for Breakout Boards"
- moved on the sheet: C1, C10, C11, C12, C13, C14, C15, C16, C17, C18, C19, C2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
